File: CPU-2/cpu-2.kicad_pcb (KiCad board)
At the start: 2 copper layers, 269.2 x 180.3 mm, 65 parts, among them X1 14-Pin Socket, X2 14-Pin Socket, X3 14-Pin Socket, X4 14-Pin Socket, X5 14-Pin Socket, X6 14-Pin Socket

Commit message: More updates to schematics, books, created RS232 interface project
Parts:
- added E25: (SPARE), Package_DIP:DIP-14_W10.16mm, F.Cu at (27.9, 110.5)
- added E30: 4N33N, Package_DIP:DIP-6_W10.16mm, F.Cu at (215.2, 67.7)
- added E31: 4N33N, Package_DIP:DIP-6_W10.16mm, F.Cu at (215.2, 76.9)
- added E40: SN7405N, Package_DIP:DIP-14_W10.16mm, F.Cu at (215.2, 48.3)
- added E41: SN7405N, Package_DIP:DIP-14_W10.16mm, F.Cu at (228.6, 48.3)
- added E46: MC1488N, Package_DIP:DIP-14_W10.16mm, F.Cu at (241.9, 48.3)
- added E52: MC1489, Package_DIP:DIP-14_W10.16mm, F.Cu at (255.3, 48.3)
Connections:
- D10 pad 1: unconnected-(D10-K-Pad1) -> Net-(D10-K)
- D10 pad 2: unconnected-(D10-A-Pad2) -> -12V
- D11 pad 1: unconnected-(D11-K-Pad1) -> Net-(D10-K)
- D11 pad 2: unconnected-(D11-A-Pad2) -> Net-(D11-A)
- D12 pad 1: unconnected-(D12-K-Pad1) -> +5V
- D12 pad 2: unconnected-(D12-A-Pad2) -> Net-(D12-A)
- E1 pad 11: Net-(E1-A5) -> /D_{3}
- E1 pad 13: unconnected-(E1-Y6-Pad13) -> /D_{1}
- E1 pad 14: unconnected-(E1-A6-Pad14) -> Net-(E1-A6)
- E1 pad 2: unconnected-(E1-A1-Pad2) -> Net-(E1-A1)
- E1 pad 3: unconnected-(E1-Y1-Pad3) -> /D_{0}
- E1 pad 4: unconnected-(E1-A2-Pad4) -> Net-(E1-A2)
- E1 pad 5: unconnected-(E1-Y3-Pad5) -> /D_{2}
- E1 pad 7: Net-(E1-A3) -> /D_{4}
- E1 pad 9: Net-(E1-Y4) -> /D_{5}
- E11 pad 6: unconnected-(E11-DI-Pad6) -> /D_{2}
- E11 pad 7: unconnected-(E11-~{DO}-Pad7) -> Net-(E1-A2)
- E17 pad 6: Net-(E17-DI) -> /D_{3}
- E19 pad 6: Net-(E19-DI) -> /D_{4}
- E2 pad 6: unconnected-(E2-DI-Pad6) -> /D_{0}
- E2 pad 7: unconnected-(E2-~{DO}-Pad7) -> Net-(E1-A1)
- E26 pad 6: Net-(E1-Y4) -> /D_{5}
- E3 pad 1: unconnected-(E3-VSS-Pad1) -> GNDREF
- E3 pad 10: unconnected-(E3-PB0-Pad10) -> Net-(E3-PB0)
- E3 pad 11: unconnected-(E3-PB1-Pad11) -> Net-(E3-PB1)
- E3 pad 12: unconnected-(E3-PB2-Pad12) -> Net-(E3-PB2)
- E3 pad 13: unconnected-(E3-PB3-Pad13) -> Net-(E3-PB3)
- E3 pad 14: unconnected-(E3-PB4-Pad14) -> Net-(E3-PB4)
- E3 pad 15: unconnected-(E3-PB5-Pad15) -> Net-(E3-PB5)
- E3 pad 16: unconnected-(E3-PB6-Pad16) -> Net-(E3-PB6)
- E3 pad 17: unconnected-(E3-PB7-Pad17) -> Net-(E3-PB7)
- E3 pad 18: unconnected-(E3-CB1-Pad18) -> Net-(E3-CB1)
- E3 pad 19: unconnected-(E3-CB2-Pad19) -> Net-(E3-CB2)
- E3 pad 2: unconnected-(E3-PA0-Pad2) -> Net-(E3-PA0)
- E3 pad 20: unconnected-(E3-V_{CC}-Pad20) -> Net-(E3-V_{CC})
- E3 pad 21: unconnected-(E3-R/~{W}-Pad21) -> /_{RW }
- E3 pad 22: unconnected-(E3-CS0-Pad22) -> /_{A6}
- E3 pad 23: unconnected-(E3-~{CS2}-Pad23) -> /_{A2}
- E3 pad 24: unconnected-(E3-CS1-Pad24) -> Net-(E24-2B)
- E3 pad 25: unconnected-(E3-ENABLE-Pad25) -> +5V
- E3 pad 26: unconnected-(E3-D7-Pad26) -> /D_{7}
- E3 pad 27: unconnected-(E3-D6-Pad27) -> /D_{6}
- E3 pad 28: unconnected-(E3-D5-Pad28) -> /D_{5}
- E3 pad 29: unconnected-(E3-D4-Pad29) -> /D_{4}
- E3 pad 3: unconnected-(E3-PA1-Pad3) -> Net-(E3-PA1)
- E3 pad 30: unconnected-(E3-D3-Pad30) -> /D_{3}
- E3 pad 31: unconnected-(E3-D2-Pad31) -> /D_{2}
- E3 pad 32: unconnected-(E3-D1-Pad32) -> /D_{1}
- E3 pad 33: unconnected-(E3-D0-Pad33) -> /D_{0}
- E3 pad 34: unconnected-(E3-~{RESET}-Pad34) -> Net-(E3-~{RESET})
- E3 pad 35: unconnected-(E3-RS1-Pad35) -> /_{A1}
- E3 pad 36: unconnected-(E3-RS0-Pad36) -> /_{A0}
- E3 pad 37: unconnected-(E3-~{IRQB}-Pad37) -> /_{~{IRQ} }
- E3 pad 38: unconnected-(E3-~{IRQA}-Pad38) -> /_{~{IRQ} }
- E3 pad 39: unconnected-(E3-CA2-Pad39) -> Net-(E3-CA2)
- E3 pad 4: unconnected-(E3-PA2-Pad4) -> Net-(E3-PA2)
- E3 pad 40: unconnected-(E3-CA1-Pad40) -> / 32
- E3 pad 5: unconnected-(E3-PA3-Pad5) -> Net-(E3-PA3)
- E3 pad 6: unconnected-(E3-PA4-Pad6) -> Net-(E3-PA4)
- E3 pad 7: unconnected-(E3-PA5-Pad7) -> Net-(E3-PA5)
- E3 pad 8: unconnected-(E3-PA6-Pad8) -> Net-(E3-PA6)
- E3 pad 9: unconnected-(E3-PA7-Pad9) -> Net-(E3-PA7)
- E33 pad 5: Net-(E36-DI) -> /D_{7}
- E33 pad 9: Net-(E33-Y4) -> /D_{6}
- E34 pad 6: Net-(E33-Y4) -> /D_{6}
- E36 pad 6: Net-(E36-DI) -> /D_{7}
- E42 pad 1: Net-(E19-DI) -> /D_{4}
- E42 pad 12: unconnected-(E42-B_{C}-Pad12) -> /D_{7}
- E42 pad 15: Net-(E1-Y4) -> /D_{5}
- E42 pad 4: Net-(E33-Y4) -> /D_{6}
- E43 pad 1: unconnected-(E43-BUS_{A}-Pad1) -> /D_{1}
- E43 pad 12: Net-(E17-DI) -> /D_{3}
- E43 pad 15: unconnected-(E43-B_{D}-Pad15) -> /D_{0}
- E43 pad 4: unconnected-(E43-BUS_{B}-Pad4) -> /D_{2}
- E5 pad 6: unconnected-(E5-DI-Pad6) -> /D_{1}
- E5 pad 7: unconnected-(E5-~{DO}-Pad7) -> Net-(E1-A6)
- E50 pad 10: unconnected-(E50-A1-Pad10) -> Net-(E48-A5)
- E50 pad 11: unconnected-(E50-A2-Pad11) -> Net-(E48-A4)
- E50 pad 12: unconnected-(E50-A3-Pad12) -> Net-(E48-A3)
- E50 pad 13: unconnected-(E50-A4-Pad13) -> Net-(E48-A2)
- E50 pad 14: unconnected-(E50-A5-Pad14) -> Net-(E48-A1)
- E50 pad 15: unconnected-(E50-A6-Pad15) -> Net-(E47-A4)
- E50 pad 16: unconnected-(E50-A7-Pad16) -> Net-(E47-A5)
- E50 pad 17: unconnected-(E50-A8-Pad17) -> Net-(E47-A6)
- E50 pad 18: unconnected-(E50-A9-Pad18) -> Net-(E47-A1)
- E50 pad 19: unconnected-(E50-A10-Pad19) -> Net-(E47-A2)
- E50 pad 2: unconnected-(E50-~{HALT}-Pad2) -> Net-(E38-1A)
- E50 pad 20: unconnected-(E50-A11-Pad20) -> Net-(E47-A3)
- E50 pad 22: unconnected-(E50-A12-Pad22) -> Net-(E44-A4)
- E50 pad 23: unconnected-(E50-A13-Pad23) -> Net-(E44-A3)
- E50 pad 24: unconnected-(E50-A14-Pad24) -> Net-(E44-A2)
- E50 pad 25: unconnected-(E50-A15-Pad25) -> Net-(E44-A1)
- E50 pad 3: unconnected-(E50-Phi1-Pad3) -> Net-(E50-Phi1)
- E50 pad 34: unconnected-(E50-R/~{W}-Pad34) -> Net-(E44-A6)
- E50 pad 39: unconnected-(E50-TSC-Pad39) -> GNDREF
- E50 pad 4: unconnected-(E50-~{IRQ}-Pad4) -> Net-(E50-~{IRQ})
- E50 pad 5: unconnected-(E50-VMA-Pad5) -> Net-(E44-A5)
- E50 pad 6: unconnected-(E50-~{NMI}-Pad6) -> Net-(E50-~{NMI})
- E50 pad 9: unconnected-(E50-A0-Pad9) -> Net-(E48-A6)
- R11 pad 1: unconnected-(R11-Pad1) -> Net-(E45-R_{ext}/C_{ext}2)
- R11 pad 2: unconnected-(R11-Pad2) -> +5V
- R12 pad 1: unconnected-(R12-Pad1) -> Net-(E45-R_{ext}/C_{ext}1)
- R12 pad 2: unconnected-(R12-Pad2) -> +5V
- R14 pad 1: unconnected-(R14-Pad1) -> Net-(E45-R_{ext}/C_{ext}2)
- R14 pad 2: unconnected-(R14-Pad2) -> +5V
- R15 pad 1: unconnected-(R15-Pad1) -> +5V
- R15 pad 2: unconnected-(R15-Pad2) -> Net-(E45-B1)
- R16 pad 1: unconnected-(R16-Pad1) -> Net-(E40-3A)
- R16 pad 2: unconnected-(R16-Pad2) -> +5V
- R17 pad 1: unconnected-(R17-Pad1) -> Net-(E40-3Y)
- R17 pad 2: unconnected-(R17-Pad2) -> +5V
- R18 pad 2: GNDREF -> Net-(E50-~{RESET})
- R2 pad 1: unconnected-(R2-Pad1) -> Net-(E8-R_{ext}/C_{ext}2)
- R2 pad 2: unconnected-(R2-Pad2) -> +5V
- R20 pad 2: unconnected-(R20-Pad2) -> Net-(E50-~{IRQ})
- R21 pad 1: unconnected-(R21-Pad1) -> Net-(E45-B1)
- R21 pad 2: unconnected-(R21-Pad2) -> Net-(C24-Pad1)
- R24 pad 1: unconnected-(R24-Pad1) -> Net-(E45-B1)
- R24 pad 2: unconnected-(R24-Pad2) -> Net-(C27-Pad1)
- R25 pad 1: unconnected-(R25-Pad1) -> Net-(E50-Phi1)
- R25 pad 2: unconnected-(R25-Pad2) -> Net-(E51-Pad7)
- R26 pad 1: unconnected-(R26-Pad1) -> Net-(E51-Pad1)
- R26 pad 2: unconnected-(R26-Pad2) -> Net-(E50-Phi1)
- R27 pad 1: unconnected-(R27-Pad1) -> Net-(E45-B2)
- R27 pad 2: unconnected-(R27-Pad2) -> Net-(C31-Pad1)
- R28 pad 1: unconnected-(R28-Pad1) -> +5V
- R28 pad 2: unconnected-(R28-Pad2) -> Net-(D12-A)
- R29 pad 2: unconnected-(R29-Pad2) -> Net-(E50-~{NMI})
- R3 pad 1: unconnected-(R3-Pad1) -> +5V
- R3 pad 2: unconnected-(R3-Pad2) -> Net-(E8-R_{ext}/C_{ext}1)
- R30 pad 1: unconnected-(R30-Pad1) -> Net-(E45-B2)
- R30 pad 2: unconnected-(R30-Pad2) -> Net-(C30-Pad1)
- R31 pad 1: unconnected-(R31-Pad1) -> +5V
- R31 pad 2: unconnected-(R31-Pad2) -> Net-(C27-Pad1)
- R32 pad 1: unconnected-(R32-Pad1) -> Net-(C31-Pad1)
- R32 pad 2: unconnected-(R32-Pad2) -> +5V
- R33 pad 1: unconnected-(R33-Pad1) -> +5V
- R33 pad 2: unconnected-(R33-Pad2) -> Net-(E45-B2)
- R4 pad 1: unconnected-(R4-Pad1) -> Net-(C12-Pad1)
- R4 pad 2: unconnected-(R4-Pad2) -> Net-(P7-Pad0)
- R5 pad 1: unconnected-(R5-Pad1) -> Net-(D10-K)
- R5 pad 2: unconnected-(R5-Pad2) -> Net-(P5-Pad0)
- R6 pad 1: unconnected-(R6-Pad1) -> +12V
- R9 pad 1: unconnected-(R9-Pad1) -> Net-(E40-6Y)
- R9 pad 2: unconnected-(R9-Pad2) -> Net-(E30-C-Pad2)
- X1 pad 1: unconnected-(X1-Pad1) -> /_{RW}
- X1 pad 10: unconnected-(X1-Pad10) -> /A_{13}
- X1 pad 11: unconnected-(X1-Pad11) -> /A_{12}
- X1 pad 12: unconnected-(X1-Pad12) -> /A_{11}
- X1 pad 13: unconnected-(X1-Pad13) -> /A_{10}
- X1 pad 14: unconnected-(X1-Pad14) -> +5V
- X1 pad 2: unconnected-(X1-Pad2) -> /A_{9}
- X1 pad 3: unconnected-(X1-Pad3) -> /_{VMA}
- X1 pad 4: unconnected-(X1-Pad4) -> /A_{14}
- X1 pad 5: unconnected-(X1-Pad5) -> /A_{15}
- X2 pad 1: unconnected-(X2-Pad1) -> /A_{2}
- X2 pad 2: unconnected-(X2-Pad2) -> /A_{4}
- X2 pad 3: unconnected-(X2-Pad3) -> /A_{3}
- X2 pad 4: unconnected-(X2-Pad4) -> /A_{5}
- X2 pad 5: unconnected-(X2-Pad5) -> /A_{6}
- X2 pad 6: unconnected-(X2-Pad6) -> /A_{7}
- X2 pad 7: unconnected-(X2-Pad7) -> /A_{8}
- X2 pad 8: unconnected-(X2-Pad8) -> /A_{0}
- X2 pad 9: unconnected-(X2-Pad9) -> /A_{1}
- X3 pad 1: unconnected-(X3-Pad1) -> /D_{4}
- X3 pad 13: unconnected-(X3-Pad13) -> /D_{5}
- X3 pad 14: unconnected-(X3-Pad14) -> /D_{6}
- X3 pad 2: unconnected-(X3-Pad2) -> /D_{7}
- X3 pad 3: unconnected-(X3-Pad3) -> /_{BA'}
- X3 pad 4: unconnected-(X3-Pad4) -> Net-(E15-Y3-Pad5)
- X3 pad 5: unconnected-(X3-Pad5) -> /D_{3}
- X3 pad 6: unconnected-(X3-Pad6) -> /D_{2}
- X3 pad 7: unconnected-(X3-Pad7) -> /D_{0}
- X3 pad 8: unconnected-(X3-Pad8) -> /D_{1}
- X3 pad 9: unconnected-(X3-Pad9) -> Net-(E29-3Y)
- X4 pad 1: unconnected-(X4-Pad1) -> Net-(E3-~{RESET})
- X4 pad 10: unconnected-(X4-Pad10) -> Net-(E3-PA4)
- X4 pad 11: unconnected-(X4-Pad11) -> Net-(E3-PA2)
- X4 pad 12: unconnected-(X4-Pad12) -> Net-(E3-CA2)
- X4 pad 2: unconnected-(X4-Pad2) -> Net-(E3-PA0)
- X4 pad 3: unconnected-(X4-Pad3) -> Net-(E3-PA1)
- X4 pad 4: unconnected-(X4-Pad4) -> Net-(E3-PA3)
- X4 pad 5: unconnected-(X4-Pad5) -> Net-(E3-PA5)
- X4 pad 6: unconnected-(X4-Pad6) -> Net-(E3-PA6)
- X4 pad 7: unconnected-(X4-Pad7) -> Net-(E3-V_{CC})
- X4 pad 8: unconnected-(X4-Pad8) -> GNDREF
- X4 pad 9: unconnected-(X4-Pad9) -> Net-(E3-PA7)
- X5 pad 1: unconnected-(X5-Pad1) -> Net-(E3-~{RESET})
- X5 pad 10: unconnected-(X5-Pad10) -> Net-(E3-PB4)
- X5 pad 11: unconnected-(X5-Pad11) -> Net-(E3-PB2)
- X5 pad 12: unconnected-(X5-Pad12) -> Net-(E3-CB2)
- X5 pad 13: unconnected-(X5-Pad13) -> Net-(E3-CB1)
- X5 pad 14: unconnected-(X5-Pad14) -> +5V
- X5 pad 2: unconnected-(X5-Pad2) -> Net-(E3-PB0)
- X5 pad 3: unconnected-(X5-Pad3) -> Net-(E3-PB1)
- X5 pad 4: unconnected-(X5-Pad4) -> Net-(E3-PB3)
- X5 pad 5: unconnected-(X5-Pad5) -> Net-(E3-PB5)
- X5 pad 6: unconnected-(X5-Pad6) -> Net-(E3-PB6)
- X5 pad 7: unconnected-(X5-Pad7) -> +5V
- X5 pad 8: unconnected-(X5-Pad8) -> GNDREF
- X5 pad 9: unconnected-(X5-Pad9) -> Net-(E3-PB7)

Commit message: Latest updates
Parts:
- added C1: CK-104, Capacitor_THT:CP_Axial_L10.0mm_D4.5mm_P15.00mm_Horizontal, F.Cu at (39.9, 42.2)
- added C10: EK47/16, Capacitor_THT:CP_Radial_D7.5mm_P2.50mm, F.Cu at (72.9, 127.9)
- added C11: EK47/16, Capacitor_THT:CP_Radial_D7.5mm_P2.50mm, F.Cu at (72.9, 136.9)
- added C12: CK-104, Capacitor_THT:CP_Axial_L10.0mm_D4.5mm_P15.00mm_Horizontal, F.Cu at (39.9, 81.4)
- added C13: EK47/16, Capacitor_THT:CP_Radial_D7.5mm_P2.50mm, F.Cu at (72.9, 146.0)
- added C14: CK-104, Capacitor_THT:CP_Axial_L10.0mm_D4.5mm_P15.00mm_Horizontal, F.Cu at (39.9, 87.9)
- added C15: CK-104, Capacitor_THT:CP_Axial_L10.0mm_D4.5mm_P15.00mm_Horizontal, F.Cu at (39.9, 94.5)
- added C16: DDM-103', Capacitor_THT:C_Disc_D10.5mm_W5.0mm_P10.00mm, F.Cu at (400.5, 286.8)
- added C17: DDM-103, Capacitor_THT:C_Disc_D10.5mm_W5.0mm_P10.00mm, F.Cu at (400.5, 293.3)
- added C18: EK47/16, Capacitor_THT:CP_Radial_D7.5mm_P2.50mm, F.Cu at (82.1, 109.8)
- added C19: CK-104, Capacitor_THT:CP_Axial_L10.0mm_D4.5mm_P15.00mm_Horizontal, F.Cu at (39.9, 101.0)
- added C2: _{EK47/16}, Capacitor_THT:CP_Radial_D7.5mm_P2.50mm, F.Cu at (72.9, 109.8)
- added C20: CK-104, Capacitor_THT:CP_Axial_L10.0mm_D4.5mm_P15.00mm_Horizontal, F.Cu at (39.9, 107.5)
- added C21: DD-101, Capacitor_THT:C_Disc_D10.5mm_W5.0mm_P10.00mm, F.Cu at (400.5, 299.9)
- added C22: DDM-103, Capacitor_THT:C_Disc_D10.5mm_W5.0mm_P10.00mm, F.Cu at (400.5, 306.4)
- added C23: DDM-103, Capacitor_THT:C_Disc_D10.5mm_W5.0mm_P10.00mm, F.Cu at (400.5, 313.0)
- added C24: DD-680, Capacitor_THT:C_Disc_D10.5mm_W5.0mm_P10.00mm, F.Cu at (400.5, 319.5)
- added C25: EK47/16, Capacitor_THT:CP_Radial_D7.5mm_P2.50mm, F.Cu at (82.1, 118.8)
- added C26: _{DDM-103'}, Capacitor_THT:C_Disc_D10.5mm_W5.0mm_P10.00mm, F.Cu at (400.5, 326.1)
- added C27: DD-101, Capacitor_THT:C_Disc_D10.5mm_W5.0mm_P10.00mm, F.Cu at (400.5, 332.6)
- added C28: EK47/16, Capacitor_THT:CP_Radial_D7.5mm_P2.50mm, F.Cu at (82.1, 127.9)
- added C29: EK47/16, Capacitor_THT:CP_Radial_D7.5mm_P2.50mm, F.Cu at (82.1, 136.9)
- added C3: EK47/16, Capacitor_THT:CP_Radial_D7.5mm_P2.50mm, F.Cu at (72.9, 118.8)
- added C30: DD-680, Capacitor_THT:C_Disc_D10.5mm_W5.0mm_P10.00mm, F.Cu at (400.5, 339.2)
- added C31: DD-101, Capacitor_THT:C_Disc_D10.5mm_W5.0mm_P10.00mm, F.Cu at (400.5, 345.7)
- added C32: EK47/16, Capacitor_THT:CP_Radial_D7.5mm_P2.50mm, F.Cu at (82.1, 146.0)
- added C4: CK-104, Capacitor_THT:CP_Axial_L10.0mm_D4.5mm_P15.00mm_Horizontal, F.Cu at (39.9, 48.7)
- added C5: Tantalum Capacitor, Capacitor_THT:CP_Axial_L18.0mm_D6.5mm_P25.00mm_Horizontal, F.Cu at (541.7, 17.3)
- added C6: CK-104, Capacitor_THT:CP_Axial_L10.0mm_D4.5mm_P15.00mm_Horizontal, F.Cu at (553.3, 19.9)
- added C7: CK-104, Capacitor_THT:CP_Axial_L10.0mm_D4.5mm_P15.00mm_Horizontal, F.Cu at (39.9, 61.8)
- added C8: CK-104, Capacitor_THT:CP_Axial_L10.0mm_D4.5mm_P15.00mm_Horizontal, F.Cu at (334.5, 154.3)
- added C9: CK-104, Capacitor_THT:CP_Axial_L10.0mm_D4.5mm_P15.00mm_Horizontal, F.Cu at (334.9, 170.5)
- added E10: SN7402N, Package_DIP:DIP-14_W10.16mm, F.Cu at (119.5, 289.6)
- added E12: MM1702A, Package_DIP:DIP-24_W10.16mm_Socket, F.Cu at (291.6, 147.9)
- added E13: SN7442N, Package_DIP:DIP-16_W7.62mm, F.Cu at (42.9, 333.8)
- added E14: SN7411N, Package_DIP:DIP-14_W10.16mm, F.Cu at (132.8, 289.6)
- added E15: DM8097N, Package_DIP:DIP-16_W7.62mm, F.Cu at (90.3, 347.8)
- added E16: SN7402N, Package_DIP:DIP-14_W10.16mm, F.Cu at (146.2, 289.6)
- added E18: SN7411N, Package_DIP:DIP-14_W10.16mm, F.Cu at (159.5, 289.6)
- added E20: MM1702A, Package_DIP:DIP-24_W10.16mm_Socket, F.Cu at (291.6, 170.7)
- added E21: DM8097N, Package_DIP:DIP-16_W7.62mm, F.Cu at (101.2, 347.8)
- added E22: SN7493N, Package_DIP:DIP-14_W10.16mm, F.Cu at (79.4, 309.0)
- added E23: SN7402N, Package_DIP:DIP-14_W10.16mm, F.Cu at (92.8, 309.0)
- added E24: SN7420N, Package_DIP:DIP-14_W10.16mm, F.Cu at (106.1, 309.0)
- added E27: SN7493N, Package_DIP:DIP-14_W10.16mm, F.Cu at (119.5, 309.0)
- added E28: SN7408N, Package_DIP:DIP-14_W10.16mm, F.Cu at (132.8, 309.0)
- added E29: SN7404N, Package_DIP:DIP-14_W10.16mm, F.Cu at (146.2, 309.0)
- added E32: SN7400N, Package_DIP:DIP-14_W10.16mm, F.Cu at (159.5, 309.0)
- added E35: MM1702A, Package_DIP:DIP-24_W10.16mm_Socket, F.Cu at (291.6, 192.2)
- added E37: SN7474N, Package_DIP:DIP-14_W10.16mm, F.Cu at (79.4, 328.4)
- added E38: SN74123N, Package_DIP:DIP-16_W10.16mm, F.Cu at (218.9, 312.4)
- added E39: SN7400N, Package_DIP:DIP-14_W10.16mm, F.Cu at (92.8, 328.4)
- added E4: SN7420N, Package_DIP:DIP-14_W10.16mm, F.Cu at (79.4, 289.6)
- added E44: DM8097N, Package_DIP:DIP-16_W7.62mm, F.Cu at (112.0, 347.8)
- added E45: DM9602N, Package_DIP:DIP-16_W7.62mm, F.Cu at (122.8, 347.8)
- added E47: DM8097N, Package_DIP:DIP-16_W7.62mm, F.Cu at (133.7, 347.8)
- added E48: DM8097N, Package_DIP:DIP-16_W7.62mm, F.Cu at (144.6, 347.8)
- added E49: SN7486N, Package_DIP:DIP-14_W10.16mm, F.Cu at (106.1, 328.4)
- added E51: MPQ6842, Package_DIP:DIP-14_W10.16mm, F.Cu at (119.5, 328.4)
- added E6: MM1702A, Package_DIP:DIP-24_W10.16mm_Socket, F.Cu at (291.3, 125.6)
- added E7: SN7493N, Package_DIP:DIP-14_W10.16mm, F.Cu at (92.8, 289.6)
- added E8: DM9602N, Package_DIP:DIP-16_W7.62mm, F.Cu at (79.5, 347.8)
- added E9: SN7474N, Package_DIP:DIP-14_W10.16mm, F.Cu at (106.1, 289.6)
- added JP1: Jumper_Open, Connector_PinHeader_1.00mm:PinHeader_1x02_P1.00mm_Vertical, F.Cu at (81.0, 54.3)
- added P1: ~, Connector_PinHeader_1.00mm:PinHeader_1x01_P1.00mm_Vertical, F.Cu at (73.5, 194.1)
- added P10: ~, Connector_PinHeader_1.00mm:PinHeader_1x01_P1.00mm_Vertical, F.Cu at (80.2, 200.2)
- added P2: ~, Connector_PinHeader_1.00mm:PinHeader_1x01_P1.00mm_Vertical, F.Cu at (73.5, 197.2)
- added P3: ~, Connector_PinHeader_1.00mm:PinHeader_1x01_P1.00mm_Vertical, F.Cu at (73.5, 200.2)
- added P5: ~, Connector_PinHeader_1.00mm:PinHeader_1x01_P1.00mm_Vertical, F.Cu at (76.9, 194.1)
- added P6: ~, Connector_PinHeader_1.00mm:PinHeader_1x01_P1.00mm_Vertical, F.Cu at (76.9, 197.2)
- added P7: ~, Connector_PinHeader_1.00mm:PinHeader_1x01_P1.00mm_Vertical, F.Cu at (76.9, 200.2)
- added P8: ~, Connector_PinHeader_1.00mm:PinHeader_1x01_P1.00mm_Vertical, F.Cu at (80.2, 194.1)
- added P9: ~, Connector_PinHeader_1.00mm:PinHeader_1x01_P1.00mm_Vertical, F.Cu at (80.2, 197.2)
- added Q1: 2N2369A, Package_TO_SOT_THT:TO-18-3_Lens, F.Cu at (467.4, 160.7)
- added TSC1: ~, Connector_PinHeader_1.00mm:PinHeader_1x02_P1.00mm_Vertical, F.Cu at (84.4, 54.3)
- added TSC10: ~, Connector_PinHeader_1.00mm:PinHeader_1x02_P1.00mm_Vertical, F.Cu at (87.7, 62.4)
- added TSC2: ~, Connector_PinHeader_1.00mm:PinHeader_1x02_P1.00mm_Vertical, F.Cu at (87.7, 54.3)
- added TSC3: ~, Connector_PinHeader_1.00mm:PinHeader_1x02_P1.00mm_Vertical, F.Cu at (91.1, 54.3)
- added TSC4: ~, Connector_PinHeader_1.00mm:PinHeader_1x02_P1.00mm_Vertical, F.Cu at (81.0, 58.4)
- added TSC5: ~, Connector_PinHeader_1.00mm:PinHeader_1x02_P1.00mm_Vertical, F.Cu at (84.4, 58.4)
- added TSC6: ~, Connector_PinHeader_1.00mm:PinHeader_1x02_P1.00mm_Vertical, F.Cu at (87.7, 58.4)
- added TSC7: ~, Connector_PinHeader_1.00mm:PinHeader_1x02_P1.00mm_Vertical, F.Cu at (91.1, 58.4)
- added TSC8: ~, Connector_PinHeader_1.00mm:PinHeader_1x02_P1.00mm_Vertical, F.Cu at (81.0, 62.4)
- added TSC9: ~, Connector_PinHeader_1.00mm:PinHeader_1x02_P1.00mm_Vertical, F.Cu at (84.4, 62.4)
- moved E40 401.6 mm to (526.3, 302.3), turned to 90 degrees
- moved E52 392.1 mm to (526.9, 331.0), turned to 90 degrees
- moved E46 390.8 mm to (526.5, 316.1), turned to 90 degrees
- moved E31 352.3 mm to (529.2, 236.6)
- moved E30 343.8 mm to (514.7, 236.5)
- moved R33 324.9 mm to (532.1, 342.4)
- moved R32 323.1 mm to (531.7, 336.7)
- moved R31 317.1 mm to (518.5, 342.3)
- moved E41 309.6 mm to (37.4, 291.7), turned to 90 degrees
- moved R12 295.8 mm to (511.5, 288.0)
- moved X6 269.8 mm to (521.2, 21.4)
- moved E50 237.9 mm to (253.9, 361.4)
- moved E3 234.5 mm to (343.6, 79.4)
- moved D6 201.1 mm to (372.5, 94.9), turned to -90 degrees
- moved D5 194.3 mm to (365.6, 94.8), turned to -90 degrees
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Connections:
- D1 pad 1: unconnected-(D1-A1-Pad1) -> GNDREF
- D1 pad 2: unconnected-(D1-A2-Pad2) -> -3V3
- D3 pad 1: unconnected-(D3-K-Pad1) -> GNDREF
- D3 pad 2: unconnected-(D3-A-Pad2) -> -3V3
- D4 pad 1: unconnected-(D4-K-Pad1) -> GNDREF
- D4 pad 2: unconnected-(D4-A-Pad2) -> Net-(D4-A)
- D5 pad 1: unconnected-(D5-K-Pad1) -> Net-(D5-K)
- D5 pad 2: unconnected-(D5-A-Pad2) -> Net-(D5-A)
- D6 pad 1: unconnected-(D6-K-Pad1) -> Net-(D6-K)
- D6 pad 2: unconnected-(D6-A-Pad2) -> Net-(D5-K)
- D7 pad 1: unconnected-(D7-K-Pad1) -> Net-(D4-A)
- D7 pad 2: unconnected-(D7-A-Pad2) -> Net-(D6-K)
- D8 pad 1: unconnected-(D8-K-Pad1) -> Net-(D5-A)
- D9 pad 1: unconnected-(D9-K-Pad1) -> +12V
- D9 pad 2: unconnected-(D9-A-Pad2) -> GNDREF
- E11 pad 1: -5V -> -3V3
- E17 pad 1: -5V -> -3V3
- E19 pad 1: -5V -> -3V3
- E2 pad 1: -5V -> -3V3
- E26 pad 1: -5V -> -3V3
- E34 pad 1: -5V -> -3V3
- E36 pad 1: -5V -> -3V3
- E41 pad 10: unconnected-(E41-5Y-Pad10) -> Net-(E32-1B)
- E41 pad 11: unconnected-(E41-5A-Pad11) -> Net-(E24-1Y)
- E41 pad 7: unconnected-(E41-GND-Pad7) -> +5V
- E5 pad 1: -5V -> -3V3
- E50 pad 7: unconnected-(E50-BA-Pad7) -> Net-(E23-3B)
- R10 pad 1: unconnected-(R10-Pad1) -> Net-(E38-1R_{ext}/C_{ext})
- R10 pad 2: unconnected-(R10-Pad2) -> +5V
- R13 pad 1: unconnected-(R13-Pad1) -> Net-(E38-2R_{ext}/C_{ext})
- R13 pad 2: unconnected-(R13-Pad2) -> +5V
- R19 pad 1: unconnected-(R19-Pad1) -> Net-(E32-1B)
- R19 pad 2: unconnected-(R19-Pad2) -> +5V
- R7 pad 1: unconnected-(R7-Pad1) -> +5V
- R7 pad 2: unconnected-(R7-Pad2) -> /_{~{HLT}}
- X6 pad 1: unconnected-(X6-Pad1) -> GNDREF
- X6 pad 10: unconnected-(X6-Pad10) -> +12V
- X6 pad 11: unconnected-(X6-Pad11) -> -3V3
- X6 pad 12: unconnected-(X6-Pad12) -> Net-(D4-A)
- X6 pad 13: unconnected-(X6-Pad13) -> +5V
- X6 pad 14: unconnected-(X6-Pad14) -> +5V
- X6 pad 2: unconnected-(X6-Pad2) -> GNDREF
- X6 pad 4: unconnected-(X6-Pad4) -> -3V3
- X6 pad 6: unconnected-(X6-Pad6) -> +5V
- X6 pad 7: unconnected-(X6-Pad7) -> +5V
- X6 pad 8: unconnected-(X6-Pad8) -> GNDREF
- X6 pad 9: unconnected-(X6-Pad9) -> GNDREF
Other:
- board size 269.2 x 180.3 mm -> 556 x 360.8 mm
