File: CPU-2/cpu-2.kicad_sch (KiCad schematic)
At the start: 156 parts, among them Q1 2N2369A, X1 14-Pin Socket, X2 14-Pin Socket, X3 14-Pin Socket, X4 14-Pin Socket, X5 14-Pin Socket, X6 14-Pin Socket

Commit message: Latest updates
Parts:
- removed C25: CK-104, symbol Sphere:CK-104
- removed R1: 100 Ohm ¼W, Resistor_THT:R_Axial_DIN0204_L3.6mm_D1.6mm_P7.62mm_Horizontal, symbol Sphere:RC07GF101
- added C25: EK47/16, Capacitor_THT:CP_Radial_D7.5mm_P2.50mm, symbol Sphere:EK47/16
- added JP1: Jumper_Open, Connector_PinHeader_1.00mm:PinHeader_1x02_P1.00mm_Vertical, symbol Sphere:Jumper_Open
- C1, C12, C14, C15, C19, C20, C4, C6, C7, C8, C9: footprint (none) -> Capacitor_THT:CP_Axial_L10.0mm_D4.5mm_P15.00mm_Horizontal
- C10, C11, C13, C18, C2, C28, C29, C3, C32: footprint (none) -> Capacitor_THT:CP_Radial_D7.5mm_P2.50mm
- C16, C17, C21, C22, C23, C24, C26, C27, C30, C31: footprint (none) -> Capacitor_THT:C_Disc_D10.5mm_W5.0mm_P10.00mm
- C5: footprint (none) -> Capacitor_THT:CP_Axial_L18.0mm_D6.5mm_P25.00mm_Horizontal
- E10, E14, E16, E18, E22, E23, E24, E27, E28, E29, E32, E37, E39, E4, E49, E51, E7, E9: footprint (none) -> Package_DIP:DIP-14_W10.16mm
- E12, E20, E35, E6: footprint (none) -> Package_DIP:DIP-24_W10.16mm_Socket
- E13, E15, E21, E44, E45, E47, E48, E8: footprint (none) -> Package_DIP:DIP-16_W7.62mm
- E38: footprint (none) -> Package_DIP:DIP-16_W10.16mm
- P1, P10, P2, P3, P4, P5, P6, P7, P8, P9: footprint (none) -> Connector_PinHeader_1.00mm:PinHeader_1x01_P1.00mm_Vertical
- TSC1, TSC10, TSC2, TSC3, TSC4, TSC5, TSC6, TSC7, TSC8, TSC9: footprint (none) -> Connector_PinHeader_1.00mm:PinHeader_1x02_P1.00mm_Vertical
Connections:
- net -5V is gone; now on net -3V3: C2.1, E11.1 (V_{BB}), E17.1 (V_{BB}), E19.1 (V_{BB}), E2.1 (V_{BB}), E25.6, E26.1 (V_{BB}), E34.1 (V_{BB}), E36.1 (V_{BB}), E5.1 (V_{BB})
- net +12V: now also C10.1, D9.1 (K), X6.10
- net +5V: now also C28.1, C5.1, E10.7 (GND), E15.9 (Y4), E16.7 (GND), E18.7 (GND), E24.2 (1B), E24.7 (GND), E32.12 (4B), E32.7 (GND), E37.1 (1~{CLR}), E37.10 (2~{PRE}), E37.12 (2D), E37.4 (1~{PRE}), E4.7 (GND), E41.7 (GND), E49.7 (GND), X6.13, X6.14, X6.6, X6.7
- net A_{0}: now also E21.13 (Y6)
- net A_{10}: now also E10.2 (1A), E4.1 (1A)
- net A_{11}: now also E10.3 (1B), E18.3 (2A), E4.2 (1B)
- net A_{12}: now also E16.11 (4A), E4.13 (2D)
- net A_{13}: now also E16.9 (3B), E4.12 (2C)
- net A_{14}: now also E16.12 (4B), E4.10 (2B)
- net A_{15}: now also E16.8 (3A), E4.9 (2A)
- net A_{1}: now also E21.9 (Y4)
- net A_{2}: now also E21.7 (Y3)
- net A_{3}: now also E10.5 (2A), E21.2 (A1), E21.3 (Y1), E22.14 (CKA), E27.11 (Q_{D})
- net A_{4}: now also E10.8 (3A), E21.11 (Y5)
- net A_{5}: now also E10.6 (2B), E21.5 (Y3)
- net A_{7}: now also E10.9 (3B)
- net A_{8}: now also E10.11 (4A), E13.15 (A)
- net A_{9}: now also E10.12 (4B), E13.14 (B)
- net D_{0}: no longer E12.4 (D0)
- net D_{1}: no longer E12.5 (D1)
- net D_{2}: no longer E12.6 (D2)
- net D_{3}: no longer E12.7 (D3)
- net D_{4}: no longer E12.8 (D4)
- net D_{5}: no longer E12.9 (D5)
- net D_{6}: no longer E12.10 (D6)
- net D_{7}: no longer E12.11 (D7)
- net GNDREF: now also C10.2, C32.2, C5.2, D1.1 (A1), D3.1 (K), D4.1 (K), D9.2 (A), E13.13 (C), X6.1, X6.2, X6.8, X6.9
- net _{RW}: now also E29.13 (6A), E32.5 (2B), E4.5 (1D)
- net _{VMA}: now also E24.1 (1A), E32.13 (4A)
- net at C32.1: now also C28.2
- net -3V3: now reaches X6.11
- net -3V3: now also D1.2 (A2), D3.2 (A), X6.4, JP1.
- net at X6.12: now also D4.2 (A), D7.1 (K)
- net at E37.11 (2CLK): now also E38.4 (1~{Q})
- net at E28.12, E37.3 (1CLK), E9.3 (1CLK): now also E15.11 (Y5), E39.12 (4B)
- net at E37.6 (1~{Q}): now also E38.1 (1A), E50.2 (~{HALT})
- net at E37.9 (2Q): now also E23.8 (3A)
- net at E16.10 (3Y): now also E24.5 (1D)
- net at E16.13 (4Y): now also E24.4 (1C)
- net at E16.4 (2Y): now also E18.2 (1B), E4.4 (1C)
- net at E16.5 (2A): now also E32.11 (4Y)
- net at E16.6 (2B): now also E4.8 (2Y)
- net at E6.24 (V_{DO}): now also E12.24 (V_{DO}), E20.24 (V_{DO}), E35.24 (V_{DO})
- net at E22.1 (CKB): now also E21.12 (A5), E22.12 (Q_{A})
- net at E22.2 (R0(1)), E22.3 (R0(2)), E27.2 (R0(1))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: now also E15.13 (Y6), E23.2 (1A)
- net at D6.1 (K): now also D7.2 (A)
- net at D6.2 (A): now also D5.1 (K)
- net at E28.10: now also E24.6 (1Y), E41.11 (5A)
- net at E28.13, E28.2, E48.1 (~{G}1)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: now also E29.10 (5Y)
- net _{~{HLT}}: now reaches E39.9 (3B), R7.2
- net at E32.3 (1Y), E38.9 (2A): now also E29.12 (6Y)
- net at E23.1 (1Y): now also E29.9 (4A), E7.14 (CKA)
- net at E23.10 (3Y): now also E23.3 (1B), E29.11 (5A)
- net at E23.9 (3B): now also E50.7 (BA)
- net at E24.10 (2B), E3.24 (CS1): now also E18.12 (1Y)
- net at E21.1 (~{G}1): now also E21.15 (~{G}2), E29.8 (4Y)
- net at E10.1 (1Y): now also E18.1 (1A)
- net at E10.10 (3Y): now also E18.9 (3A)
- net at E10.4 (2Y): now also E18.10 (3B)
- net at E4.6 (1Y): now also E13.12 (D)
- net at D5.2 (A): now also D8.1 (K)
- net at E18., E18.8 (3Y): now also E18.13 (1C)
- new net _{D_{0}}: E12.4 (D0)
- new net _{D_{1}}: E12.5 (D1)
- new net _{D_{2}}: E12.6 (D2)
- new net _{D_{3}}: E12.7 (D3)
- new net _{D_{4}}: E12.8 (D4)
- new net _{D_{5}}: E12.9 (D5)
- new net _{D_{6}}: E12.10 (D6)
- new net _{D_{7}}: E12.11 (D7)
Other:
- note added: "15-JAN-1976 G.W Hone Sphere Original"
- note added: "A"
- note added: "Based on CPU/2 schematic drawn & authorised by G.W. Hone/M.Tyler 22-DEC-1975 - 15-JAN-1976"
- note added: "C"
- note added: "D"
- note added: "F"
- note added: "PLACEMENT IDENTIFIED"
- note added: "R1"
- note added: "R1 is ommitted from this schematic, as it is not present on a sample CPU/2 board."
- note added: "The original schematic separates chip pins out for ease of diagramming. This version does not."
- note added: "This schematic includes the RS232 interface, which is not the default on the CPU/2 board."
- note added: "~-10V NEG BIAS"
- note removed: "The original schematic separates chip pins out for ease of diagramming. This version does not"
- note removed: "This schematic includes the RS232 interface, which is not the default on the CPU/2 board"
- moved on the sheet: C10, C14, C15, C17, C20, C32, C4, C5, C6, C7, D2, D4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
