File: ORB/ORB/orb/orb.kicad_sch (KiCad schematic)
At the start: 6 parts, among them J1 Conn_01x14_Pin-1-14, J2 Conn_01x14_Pin-1-14, U1 Arduino_Nano

Commit message: Latest updates
Parts:
- removed E35/C1, E6/C1, J1, J2: Conn_01x14_Pin-1-14, symbol Project-ORB:Conn_01x14_Pin-1-14
- removed E6/C2: Conn_01x14_Pin-15-28, symbol Project-ORB:Conn_01x14_Pin-15-28
- added D1: 1N4001, Diode_THT:D_DO-41_SOD81_P10.16mm_Horizontal, symbol Sphere:1N4001
- added E12, E20, E35, E6: MM1702A, Package_DIP:DIP-24_W10.16mm_Socket, symbol Sphere:MM1702A
- added J1, J2, J3, J4: Conn_01x02_Socket, Connector_PinHeader_1.00mm:PinHeader_1x02_P1.00mm_Vertical, symbol Connector:Conn_01x02_Socket
- added U3: 4071, Connector_PinSocket_1.27mm:PinSocket_2x07_P1.27mm_Vertical, symbol Project-ORB:4071
Connections:
- net at U1.21 (A2/D16): now also E12.10 (D6), E20.10 (D6), E35.10 (D6), E6.10 (D6)
- net at U1.1 (D1/TX): now also J2.2 (Pin_2)
- net at U1.10 (D7): now also E12.1 (A2), E20.1 (A2), E35.1 (A2), E6.1 (A2)
- net at U1.11 (D8): now also E12.2 (A1), E20.2 (A1), E35.2 (A1), E6.2 (A1)
- net at U1.12 (~D9): now also E12.3 (A0), E20.3 (A0), E35.3 (A0), E6.3 (A0)
- net at U1.13 (~D10): now also E12.4 (D0), E20.4 (D0), E35.4 (D0), E6.4 (D0)
- net at U1.14 (~D11): now also E12.5 (D1), E20.5 (D1), E35.5 (D1), E6.5 (D1)
- net at U1.15 (D12): now also E12.6 (D2), E20.6 (D2), E35.6 (D2), E6.6 (D2)
- net at U1.16 (D13): now also E12.7 (D3), E20.7 (D3), E35.7 (D3), E6.7 (D3)
- net at U1.19 (A0/D14): now also E12.8 (D4), E20.8 (D4), E35.8 (D4), E6.8 (D4)
- net at U1.2 (D0/RX): now also J2.1 (Pin_1)
- net at U1.20 (A1/D15): now also E12.9 (D5), E20.9 (D5), E35.9 (D5), E6.9 (D5)
- net at U1.22 (A3/D17): now also E12.11 (D7), E20.11 (D7), E35.11 (D7), E6.11 (D7)
- net at U1.23 (A4/D18): now also J3.2 (Pin_2)
- net at U1.24 (A5/D19): now also J3.1 (Pin_1)
- net at U1.25 (A6/D20): now also U3.4
- net at U1.26 (A7/D21): now also U3.3
- net at U1.29 (GND): now also J1.2 (Pin_2)
- net at U1.30 (VIN): now also J1.1 (Pin_1)
- net at U1.5 (D2): now also E12.17 (A7), E20.17 (A7), E35.17 (A7), E6.17 (A7)
- net at U1.6 (~D3): now also E12.18 (A6), E20.18 (A6), E35.18 (A6), E6.18 (A6)
- net at U1.7 (D4): now also E12.19 (A5), E20.19 (A5), E35.19 (A5), E6.19 (A5)
- net at U1.8 (~D5): now also E12.20 (A4), E20.20 (A4), E35.20 (A4), E6.20 (A4)
- net at U1.9 (~D6): now also E12.21 (A3), E20.21 (A3), E35.21 (A3), E6.21 (A3)
- new net: D1.2 (A), E12.24 (V_{DO}), E20.24 (V_{DO}), E35.24 (V_{DO}), E6.24 (V_{DO}), J4.2 (Pin_2)
- new net: E20.14 (~{CS}), U3.1
- new net: E12.14 (~{CS}), U3.5
- new net: E6.14 (~{CS}), U3.2, U3.6
- new net: D1.1 (K), J4.1 (Pin_1)
Other:
- note added: "+5V"
- note added: "-10V -ve BIAS"
- note added: "-12V"
- note added: "Address Bus"
- note added: "Chip Select"
- note added: "Data Bus"
- note added: "EPROM 1"
- note added: "EPROM 2"
- note added: "EPROM 3"
- note added: "EPROM 4"
- note added: "EXP2-A"
- note added: "EXP2-B"
- note added: "Expansion"
- note added: "GND"
- note added: "Ground/Power"
- note added: "KEY"
- note added: "RX"
- note added: "TX"
- moved on the sheet: U1
