File: RS232/rs232/rs232/rs232.kicad_pcb (KiCad board)
At the start: 2 copper layers, 60 x 60 mm, 25 parts, among them J1 Conn_01x03_Pin, J2 Conn_01x04_Pin, J3 Conn_01x03_Pin, J4 Conn_01x02_Pin, J5 Conn_01x04_Pin

Commit message: Latest updates
Parts:
- removed the G*** at (189.8, 99.1)
- removed R17: 1 kOhm ¼W, Resistor_THT:R_Axial_DIN0204_L3.6mm_D1.6mm_P7.62mm_Horizontal
- added G***: LOGO, RS232:rs232-module-1-logo, F.Cu at (96.4, 265.7)
- added G***: LOGO, RS232:sphere-corp-board-logo, F.Cu at (96.2, 257.3)
- added G***: LOGO, RS232:rs232-module-1-logo, F.Cu at (81.3, 37.9)
- G***: moved to B.Cu
- moved J1 134.8 mm to (102.5, 86.2), turned to 90 degrees
- moved R16 133.7 mm to (102.9, 70.4)
- moved G*** 132.2 mm to (121.6, 64.9)
- moved R9 131.5 mm to (102.9, 68.0)
- moved G*** 131.3 mm to (121.8, 73.3)
- moved J3 126.2 mm to (109.4, 86.3), turned to 90 degrees
- moved R5 124.4 mm to (102.9, 65.5)
- moved TSC3 124.2 mm to (120.9, 34.8)
- moved R4 124.2 mm to (102.9, 63.2)
- moved E46 123.8 mm to (88.6, 37.9)
- moved E30 123.8 mm to (97.9, 66.2)
- moved TSC1 123.8 mm to (120.9, 46.6)
- moved TSC4 123.8 mm to (120.9, 52.6)
- moved E52 123.8 mm to (103.7, 37.9)
- moved J2 123.8 mm to (99.0, 86.2)
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Connections:
- R9 pad 1: Net-(J5-Pin_3) -> Net-(E30-C-Pad2)
- R9 pad 2: Net-(E30-C-Pad2) -> Net-(J5-Pin_3)
Routing:
- net Net-(J4-Pin_2): track 11.8 -> 87.6 mm
- net Net-(J4-Pin_1): track 13.3 -> 69.7 mm
- net Net-(J5-Pin_2): track 156.4 -> 109.2 mm, vias 0 -> 2
- net Net-(E31-E): track 114.2 -> 68.4 mm
- net Net-(J5-Pin_3): track 63.2 -> 95.0 mm
- net Net-(J5-Pin_4): track 55.9 -> 84.2 mm, vias 1 -> 0
- net Net-(D11-A): track 50.7 -> 25.0 mm
- net Net-(E46-2Y): track 38.8 -> 63.5 mm
- net Net-(E52-1A): track 41.0 -> 64.1 mm
- net Net-(E30-C-Pad2): track 34.8 -> 13.8 mm
- net Net-(J1-Pin_1): track 15.0 -> 36.1 mm
- net Net-(J1-Pin_3): track 11.6 -> 28.0 mm
- net Net-(D10-A): track 127.6 -> 118.9 mm
- net Net-(E30-A): track 53.7 -> 47.0 mm, vias 4 -> 2
- net Net-(D10-K): track 58.0 -> 64.5 mm
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Other:
- board size 60 x 60 mm -> 53.9 x 58.4 mm
- board text added: "12"
- board text added: "13"
- board text added: "5"
- board text added: "6"
- board text added: "Connect to E40 on CPU/2 board"
- board text added: "Designed and built by Andrew Shapton alshapton@gmail.com"
- board text added: "Parts List C12 0.1µF D10/D11 IN4001 x 2 E30/E31 4N33N x 2 E46 MC1488N E52 MC1489 R4 1.1KΩ 1W R5 820Ω 1W R9 2.2KΩ 1W R16 512Ω Jumpers x 2 PB0/PB7 Connectors: 2 x 1 J4 3 x 2 J1/J3 4 x 2 J2/J5 Sockets: 14 Pin x 2 6 Pin x 2"
- board text added: "Pins:"
- board text removed: "1KΩ"
- board text removed: "Connect to E40 as shown on CPU/2 board"
- board text removed: "Parts List C12 0.1µF D10/D11 IN4001 x 2 E30/E31 4N33N x 2 E46 MC1488N E52 MC1489 R4 1.1KΩ 1W R5 820Ω 1W R9 2.2KΩ 1W R16 512Ω R17 1KΩ Jumpers x 2 PB0/PB7 Connectors: 2 x 1 J4 3 x 2 J1/J3 4 x 2 J2/J5"
- board text removed: "Pins: 5 6 12 13"
