File: RS232/rs232/rs232/rs232.kicad_sch (KiCad schematic)
At the start: 21 parts, among them J1 Conn_01x03_Pin, J2 Conn_01x04_Pin, J3 Conn_01x03_Pin, J4 Conn_01x02_Pin, J5 Conn_01x04_Pin

Commit message: Latest updates
Parts:
- removed R17: 1 kOhm ¼W, Resistor_THT:R_Axial_DIN0204_L3.6mm_D1.6mm_P7.62mm_Horizontal, symbol Sphere:RC07GF102
Connections:
- net at J5.3 (Pin_3): now also R9.2; no longer R9.1
- net at E30.2 (C): now also R9.1; no longer R9.2
Other:
- note added: "0.1 10-MAY-2023 Andrew Shapton Initial Version"
- note added: "NOTES"
- note added: "REVISION HISTORY"
- note added: "The original schematic separates chip pins out for ease of diagramming. This version does not"
- moved on the sheet: C12, D10, D11, E30, E31, E46, E52, J1, J2, J3, J4, J5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
